File: Hardware/Arm Control Board/Arm Control Board.sch (KiCad schematic (older format))
At the start: 0 parts

Commit message: Added regulator to schematic
Also added gitignore, parts list, and microcontroller datasheet
Parts:
- added 100, C?: CP1, symbol CP1
- added 3k: R, symbol R
- added C?: 470 pF, symbol C
- added D?: 1N5819, symbol DIODESCH
- added L?: 220 uH, symbol INDUCTOR_SMALL
- added P?: RS485, symbol RS485
- added R?: 1k, symbol R
- added R?: .33???, symbol R
- added U?: STM32F410RCT6, symbol STM32F410RCT6
- added U?: ST485CDR, symbol ST485CDR
- added U?: AZ34063UMTR-G1, symbol AZ34063UMTR-G1
Connections:
- net labels added: +12V, GND
- wire segments 0 -> 32
