File: Hardware/Arm Control Board/Arm Control Board.kicad_pcb (KiCad board)
At the start: 2 copper layers, 0 parts

Commit message: Initial PCB layout
Parts:
- added C1: 4.7uF, Capacitors_SMD:C_1206_HandSoldering, F.Cu at (142.0, 155.5)
- added C10: .1uF, Capacitors_SMD:C_1206_HandSoldering, F.Cu at (112.0, 155.5)
- added C11: .1uF, Capacitors_SMD:C_1206_HandSoldering, F.Cu at (128.0, 155.5)
- added C12: 1uF, Capacitors_SMD:C_1206_HandSoldering, F.Cu at (134.0, 155.5)
- added C13: 10uF, Capacitors_SMD:C_1206_HandSoldering, F.Cu at (30.5, 103.5)
- added C14: 10uF, Capacitors_SMD:C_1206_HandSoldering, F.Cu at (27.0, 172.0)
- added C15: 10nF, Capacitors_SMD:C_1206_HandSoldering, F.Cu at (46.0, 87.5)
- added C16: 10nF, Capacitors_SMD:C_1206_HandSoldering, F.Cu at (46.0, 147.0)
- added C17: 4.7uF, Capacitors_SMD:C_1206_HandSoldering, F.Cu at (198.0, 63.0)
- added C18: 4.7uF, Capacitors_SMD:C_1206_HandSoldering, F.Cu at (90.0, 46.0)
- added C19: 18pF, Capacitors_SMD:C_1206_HandSoldering, F.Cu at (39.0, 29.5)
- added C2: 15pF, Capacitors_SMD:C_1206_HandSoldering, F.Cu at (99.5, 140.0)
- added C20: 18pF, Capacitors_SMD:C_1206_HandSoldering, F.Cu at (118.0, 36.0)
- added C21: 1uF, Capacitors_SMD:C_1206_HandSoldering, F.Cu at (68.0, 47.5)
- added C22: 1uF, Capacitors_SMD:C_1206_HandSoldering, F.Cu at (126.5, 60.5)
- added C23: 8.2nF, Capacitors_SMD:C_1206_HandSoldering, F.Cu at (68.0, 28.5)
- added C24: 8.2nF, Capacitors_SMD:C_1206_HandSoldering, F.Cu at (126.5, 53.5)
- added C25: 22uF, Capacitors_SMD:C_1206_HandSoldering, F.Cu at (68.0, 41.0)
- added C26: 22uF, Capacitors_SMD:C_1206_HandSoldering, F.Cu at (126.5, 32.5)
- added C27: 10uF, Capacitors_SMD:C_1206_HandSoldering, F.Cu at (68.0, 61.0)
- added C28: 22uF, Capacitors_SMD:C_1206_HandSoldering, F.Cu at (68.0, 34.5)
- added C29: 10uF, Capacitors_SMD:C_1206_HandSoldering, F.Cu at (126.5, 39.5)
- added C3: .1uF, Capacitors_SMD:C_1206_HandSoldering, F.Cu at (67.5, 155.5)
- added C30: 22uF, Capacitors_SMD:C_1206_HandSoldering, F.Cu at (126.5, 25.5)
- added C31: .1uF, Capacitors_SMD:C_1206_HandSoldering, F.Cu at (31.0, 38.0)
- added C32: .1uF, Capacitors_SMD:C_1206_HandSoldering, F.Cu at (96.0, 46.0)
- added C33: 10uF, Capacitors_SMD:C_1206_HandSoldering, F.Cu at (68.0, 54.0)
- added C34: 10uF, Capacitors_SMD:C_1206_HandSoldering, F.Cu at (126.5, 46.5)
- added C35: 18pF, Capacitors_SMD:C_1206_HandSoldering, F.Cu at (179.0, 22.0)
- added C36: 18pF, Capacitors_SMD:C_1206_HandSoldering, F.Cu at (231.5, 24.5)
- added C37: 1uF, Capacitors_SMD:C_1206_HandSoldering, F.Cu at (198.0, 38.0)
- added C38: 1uF, Capacitors_SMD:C_1206_HandSoldering, F.Cu at (250.5, 35.0)
- added C39: 8.2nF, Capacitors_SMD:C_1206_HandSoldering, F.Cu at (198.0, 44.5)
- added C4: .1uF, Capacitors_SMD:C_1206_HandSoldering, F.Cu at (74.5, 155.5)
- added C40: 8.2nF, Capacitors_SMD:C_1206_HandSoldering, F.Cu at (250.5, 41.5)
- added C41: 22uF, Capacitors_SMD:C_1206_HandSoldering, F.Cu at (165.5, 24.0)
- added C42: 22uF, Capacitors_SMD:C_1206_HandSoldering, F.Cu at (250.5, 17.0)
- added C43: 10uF, Capacitors_SMD:C_1206_HandSoldering, F.Cu at (198.0, 50.5)
- added C44: 22uF, Capacitors_SMD:C_1206_HandSoldering, F.Cu at (172.5, 24.0)
- added C45: 10uF, Capacitors_SMD:C_1206_HandSoldering, F.Cu at (250.5, 47.5)
- added C46: 22uF, Capacitors_SMD:C_1206_HandSoldering, F.Cu at (250.5, 23.0)
- added C47: .1uF, Capacitors_SMD:C_1206_HandSoldering, F.Cu at (153.5, 41.0)
- added C48: .1uF, Capacitors_SMD:C_1206_HandSoldering, F.Cu at (218.0, 36.0)
- added C49: 10uF, Capacitors_SMD:C_1206_HandSoldering, F.Cu at (198.0, 56.5)
- added C5: 15pF, Capacitors_SMD:C_1206_HandSoldering, F.Cu at (109.0, 140.0)
- added C50: 10uF, Capacitors_SMD:C_1206_HandSoldering, F.Cu at (250.5, 54.0)
- added C6: .1uF, Capacitors_SMD:C_1206_HandSoldering, F.Cu at (81.5, 155.5)
- added C7: 4.7uF, Capacitors_SMD:C_1206_HandSoldering, F.Cu at (90.0, 155.5)
- added C8: .1uF, Capacitors_SMD:C_1206_HandSoldering, F.Cu at (97.5, 155.5)
- added C9: .1uF, Capacitors_SMD:C_1206_HandSoldering, F.Cu at (105.0, 155.5)
- added FB1: 50O, Resistors_SMD:R_1206_HandSoldering, F.Cu at (119.5, 153.5)
- added L3: 3.3uH, Inductors_NEOSID:Neosid_Inductor_SM-PIC0612H, F.Cu at (31.0, 26.0)
- added L4: 3.3uH, Inductors_NEOSID:Neosid_Inductor_SM-PIC0612H, F.Cu at (107.0, 23.0)
- added L5: 3.3uH, Inductors_NEOSID:Neosid_Inductor_SM-PIC0612H, F.Cu at (156.5, 22.0)
- added L6: 3.3uH, Inductors_NEOSID:Neosid_Inductor_SM-PIC0612H, F.Cu at (221.0, 18.5)
- added R1: 49.9k, Resistors_SMD:R_1206_HandSoldering, F.Cu at (28.5, 96.5)
- added R10: 100k, Resistors_SMD:R_1206_HandSoldering, F.Cu at (116.0, 46.5)
- added R11: 191k, Resistors_SMD:R_1206_HandSoldering, F.Cu at (179.0, 16.0)
- added R12: 191k, Resistors_SMD:R_1206_HandSoldering, F.Cu at (231.5, 18.5)
- added R13: 22.1k, Resistors_SMD:R_1206_HandSoldering, F.Cu at (198.0, 31.5)
- added R14: 22.1k, Resistors_SMD:R_1206_HandSoldering, F.Cu at (250.5, 29.0)
- added R15: 100k, Resistors_SMD:R_1206_HandSoldering, F.Cu at (171.5, 49.5)
- added R16: 100k, Resistors_SMD:R_1206_HandSoldering, F.Cu at (230.5, 43.5)
- added R2: 9.53k, Resistors_SMD:R_1206_HandSoldering, F.Cu at (35.0, 96.5)
- added R3: 49.9k, Resistors_SMD:R_1206_HandSoldering, F.Cu at (37.5, 168.5)
- added R4: 15.8k, Resistors_SMD:R_1206_HandSoldering, F.Cu at (37.5, 176.0)
- added R5: 191k, Resistors_SMD:R_1206_HandSoldering, F.Cu at (39.0, 23.0)
- added R6: 191k, Resistors_SMD:R_1206_HandSoldering, F.Cu at (112.0, 30.0)
- added R7: 22.1k, Resistors_SMD:R_1206_HandSoldering, F.Cu at (68.0, 22.0)
- added R8: 22.1k, Resistors_SMD:R_1206_HandSoldering, F.Cu at (118.0, 15.0)
- added R9: 100k, Resistors_SMD:R_1206_HandSoldering, F.Cu at (46.5, 46.0)
- added U1: STM32F401RCT6, Housings_QFP:LQFP-64_10x10mm_Pitch0.5mm, F.Cu at (106.5, 98.0)
- added U2: SN75176BDR, SMD_Packages:SOIC-8-W, F.Cu at (127.5, 96.5)
- added U3: 74LVCH244APW, MAVRIC_footprints:AB2_TSSOP20, F.Cu at (121.5, 74.5)
- added U4: AOZ1280CI, SMD_Packages:SOT-23-6, F.Cu at (46.0, 98.5)
- added U5: AOZ1280CI, SMD_Packages:SOT-23-6, F.Cu at (46.0, 157.0)
- added U6: AP65552SP-13, SMD_Packages:SOIC-8-N-1EP, F.Cu at (46.5, 39.5)
- added U7: AP65552SP-13, SMD_Packages:SOIC-8-N-1EP, F.Cu at (106.0, 37.0)
- added U8: AP65552SP-13, SMD_Packages:SOIC-8-N-1EP, F.Cu at (172.5, 39.5)
- added U9: AP65552SP-13, SMD_Packages:SOIC-8-N-1EP, F.Cu at (231.0, 34.5)
- added X1: 24MHz, Crystals_Oscillators_SMD:Q_49U3HMS, F.Cu at (104.5, 131.5)

Commit message: Fixed parts with pin numbers starting at zero
just a zero indexed man living in a one indexed world
Parts:
- added D1, D2: DIODESCH, MAVRIC_footprints:Diode_MicroSMP, F.Cu at (0.00, 0.00)
- added L1, L2: 2.2uH, MAVRIC_footprints:Yuden_SMD_Power_Inductor_6060, F.Cu at (0.00, 0.00)
- added P1: Servo 1, MAVRIC_footprints:1x3_SMD_header, F.Cu at (0.00, 0.00)
- added P10: UIM240XX_Stepper_Conn, MAVRIC_footprints:1x6_SMD_header, F.Cu at (0.00, 0.00)
- added P11: Battery, MAVRIC_footprints:SolderWirePad_2x_2-5mmDrill, F.Cu at (94.5, 184.0)
- added P12: SyRen, MAVRIC_footprints:1x2_SMD_header, F.Cu at (0.00, 0.00)
- added P13: Raspberry Pi, MAVRIC_footprints:1x2_SMD_header, F.Cu at (0.00, 0.00)
- added P2: Shoulder Feedback, MAVRIC_footprints:1x3_SMD_header, F.Cu at (0.00, 0.00)
- added P3: Servo 2, MAVRIC_footprints:1x3_SMD_header, F.Cu at (0.00, 0.00)
- added P4: Servo 3, MAVRIC_footprints:1x3_SMD_header, F.Cu at (0.00, 0.00)
- added P5: Elbow Feedback, MAVRIC_footprints:1x3_SMD_header, F.Cu at (0.00, 0.00)
- added P6: Servo 4, MAVRIC_footprints:1x3_SMD_header, F.Cu at (0.00, 0.00)
- added P7: RS485, MAVRIC_footprints:1x2_SMD_header, F.Cu at (0.00, 0.00)
- added P8: ST_SWD_Connector, MAVRIC_footprints:1x6_SMD_header, F.Cu at (0.00, 0.00)
- added P9: Servo 5, MAVRIC_footprints:1x3_SMD_header, F.Cu at (0.00, 0.00)
Other:
- board outline added: 251.5 x 182.5 mm

Commit message: reg1 layout made
expecting it to change bunches
Parts:
- moved D2 347.7 mm to (347.0, 21.8)
- moved D1 347.3 mm to (347.0, 14.3)
- moved L2 337.5 mm to (337.0, 17.0)
- moved L1 330.3 mm to (329.9, 17.0)
- moved P13 300.7 mm to (256.5, 157.0), turned to 180 degrees
- moved P9 294.5 mm to (255.5, 146.5), turned to 180 degrees
- moved P6 290.4 mm to (255.5, 138.0), turned to 180 degrees
- moved P4 286.4 mm to (255.5, 129.5), turned to 180 degrees
- moved P3 282.7 mm to (255.5, 121.0), turned to 180 degrees
- moved P1 279.2 mm to (255.5, 112.5), turned to 180 degrees
- moved P12 272.5 mm to (255.0, 96.0), turned to 270 degrees
- moved P10 264.7 mm to (252.0, 81.0)
- moved P5 250.1 mm to (236.5, 81.5), turned to 270 degrees
- moved P2 241.2 mm to (227.0, 81.5), turned to 270 degrees
- moved R5 221.1 mm to (242.8, 108.8)
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Routing:
- net /7.4V Regulators/REG1+7V4: track 0.00 -> 31.9 mm
- net GND: track 0.00 -> 29.7 mm
- net Net-(C19-Pad2): track 0.00 -> 26.2 mm
- net +12V: track 0.00 -> 15.9 mm
- net Net-(C31-Pad2): track 0.00 -> 14.9 mm
- net Net-(C21-Pad1): track 0.00 -> 7.72 mm
- net Net-(C31-Pad1): track 0.00 -> 4.40 mm
- net /7.4V Regulators/REG1EN: track 0.00 -> 3.87 mm
- net Net-(C23-Pad1): track 0.00 -> 3.37 mm
Other:
- board outline removed

Commit message: started reg2 layout
Parts:
- moved C18 250.7 mm to (-59.2, 170.8), turned to 180 degrees
- moved R6 225.0 mm to (243.2, 141.2)
- moved C30 223.1 mm to (243.2, 143.8)
- moved C22 220.1 mm to (243.2, 175.2)
- moved C24 220.1 mm to (243.2, 168.2)
- moved L4 220.1 mm to (223.8, 137.8)
- moved R8 220.1 mm to (234.8, 129.8)
- moved U7 220.1 mm to (222.8, 151.8)
- moved C26 219.3 mm to (243.2, 146.2)
- moved C29 215.8 mm to (243.2, 149.2)
- moved C32 214.8 mm to (216.8, 152.0)
- moved C20 214.6 mm to (243.2, 138.8), turned to 0 degrees
- moved C34 212.0 mm to (243.2, 151.8)
- moved R10 210.8 mm to (222.8, 156.2), turned to 180 degrees
Changed lines of the file:
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@@
     (pad_to_mask_clearance 0)
     (aux_axis_origin 0 0)
-    (visible_elements 7FFCFF7F)
+    (visible_elements 7FFEFF7F)
     (pcbplotparams
       (layerselection 0x00030_80000001)
@@
   )
   (module Capacitors_SMD:C_1206_HandSoldering (layer F.Cu)
-    (at 93.5 -28 90)
+    (at -59.25 170.75 180)
     (descr "Capacitor SMD 1206, hand soldering")
     (tags "capacitor 1206")
     (attr smd)
-    (fp_text reference C18 (at 0 -2.3 90) (layer F.SilkS)
+    (fp_text reference C18 (at 0 -2.3 180) (layer F.SilkS)
       (effects (font (size 1 1) (thickness 0.15)))
     )
-    (fp_text value 4.7uF (at 0 2.3 90) (layer F.SilkS)
+    (fp_text value 4.7uF (at 0 2.3 180) (layer F.SilkS)
       (effects (font (size 1 1) (thickness 0.15)))
     )
@@
     (fp_line (start 1 -1.025) (end -1 -1.025) (layer F.SilkS) (width 0.15))
     (fp_line (start -1 1.025) (end 1 1.025) (layer F.SilkS) (width 0.15))
-    (pad 1 smd rect (at -2 0 90) (size 2 1.6) (layers F.Cu F.Paste F.Mask)
+    (pad 1 smd rect (at -2 0 180) (size 2 1.6) (layers F.Cu F.Paste F.Mask)
       (net 12 +12V))
-    (pad 2 smd rect (at 2 0 90) (size 2 1.6) (layers F.Cu F.Paste F.Mask)
+    (pad 2 smd rect (at 2 0 180) (size 2 1.6) (layers F.Cu F.Paste F.Mask)
       (net 2 GND))
     (model Capacitors_SMD/C_1206_HandSoldering.wrl
@@
   )
   (module Capacitors_SMD:C_1206_HandSoldering (layer F.Cu)
-    (at 121.5 -38 180)
+    (at 243.25 138.75)
     (descr "Capacitor SMD 1206, hand soldering")
     (tags "capacitor 1206")
     (attr smd)
-    (fp_text reference C20 (at 0 -2.3 180) (layer F.SilkS)
+    (fp_text reference C20 (at 0 -2.3) (layer F.SilkS)
       (effects (font (size 1 1) (thickness 0.15)))
     )
-    (fp_text value 18pF (at 0 2.3 180) (layer F.SilkS)
+    (fp_text value 18pF (at 0 2.3) (layer F.SilkS)
       (effects (font (size 1 1) (thickness 0.15)))
     )
@@
     (fp_line (start 1 -1.025) (end -1 -1.025) (layer F.SilkS) (width 0.15))
     (fp_line (start -1 1.025) (end 1 1.025) (layer F.SilkS) (width 0.15))
-    (pad 1 smd rect (at -2 0 180) (size 2 1.6) (layers F.Cu F.Paste F.Mask)
+    (pad 1 smd rect (at -2 0) (size 2 1.6) (layers F.Cu F.Paste F.Mask)
       (net 15 "/7.4V Regulators/REG2+7V4"))
-    (pad 2 smd rect (at 2 0 180) (size 2 1.6) (layers F.Cu F.Paste F.Mask)
+    (pad 2 smd rect (at 2 0) (size 2 1.6) (layers F.Cu F.Paste F.Mask)
       (net 16 "Net-(C20-Pad2)"))
     (model Capacitors_SMD/C_1206_HandSoldering.wrl
@@
   )
   (module Capacitors_SMD:C_1206_HandSoldering (layer F.Cu)
-    (at 130 -13.5)
+    (at 243.25 175.25)
     (descr "Capacitor SMD 1206, hand soldering")
     (tags "capacitor 1206")
@@
   )
   (module Capacitors_SMD:C_1206_HandSoldering (layer F.Cu)
-    (at 130 -20.5)
+    (at 243.25 168.25)
     (descr "Capacitor SMD 1206, hand soldering")
     (tags "capacitor 1206")
@@
   )
   (module Capacitors_SMD:C_1206_HandSoldering (layer F.Cu)
-    (at 130 -41.5)
+    (at 243.25 146.25)
     (descr "Capacitor SMD 1206, hand soldering")
     (tags "capacitor 1206")
@@
   )
   (module Capacitors_SMD:C_1206_HandSoldering (layer F.Cu)
-    (at 130 -34.5)
+    (at 243.25 149.25)
     (descr "Capacitor SMD 1206, hand soldering")
     (tags "capacitor 1206")
@@
   )
   (module Capacitors_SMD:C_1206_HandSoldering (layer F.Cu)
-    (at 130 -48.5)
+    (at 243.25 143.75)
     (descr "Capacitor SMD 1206, hand soldering")
     (tags "capacitor 1206")
@@
   )
   (module Capacitors_SMD:C_1206_HandSoldering (layer F.Cu)
-    (at 99.5 -28 90)
+    (at 216.75 152 90)
     (descr "Capacitor SMD 1206, hand soldering")
     (tags "capacitor 1206")
@@
   )
   (module Capacitors_SMD:C_1206_HandSoldering (layer F.Cu)
-    (at 130 -27.5)
+    (at 243.25 151.75)
     (descr "Capacitor SMD 1206, hand soldering")
     (tags "capacitor 1206")
@@
   )
   (module Inductors_NEOSID:Neosid_Inductor_SM-PIC0612H (layer F.Cu)
-    (at 110.5 -51)
+    (at 223.75 137.75)
     (descr "Neosid, Power Inductor, SM-PIC0612H, Festinduktivitaet, SMD,")
     (tags "Neosid, Power Inductor, SM-PIC0612H, Festinduktivitaet, SMD,")
@@
   )
   (module Resistors_SMD:R_1206_HandSoldering (layer F.Cu)
-    (at 115.5 -44)
+    (at 243.25 141.25)
     (descr "Resistor SMD 1206, hand soldering")
     (tags "resistor 1206")
@@
   )
   (module Resistors_SMD:R_1206_HandSoldering (layer F.Cu)
-    (at 121.5 -59)
+    (at 234.75 129.75)
     (descr "Resistor SMD 1206, hand soldering")
     (tags "resistor 1206")
@@
   )
   (module Resistors_SMD:R_1206_HandSoldering (layer F.Cu)
-    (at 119.5 -27.5)
+    (at 222.75 156.25 180)
     (descr "Resistor SMD 1206, hand soldering")
     (tags "resistor 1206")
     (attr smd)
-    (fp_text reference R10 (at 0 -2.3) (layer F.SilkS)
+    (fp_text reference R10 (at 0 -2.3 180) (layer F.SilkS)
       (effects (font (size 1 1) (thickness 0.15)))
     )
-    (fp_text value 100k (at 0 2.3) (layer F.SilkS)
+    (fp_text value 100k (at 0 2.3 180) (layer F.SilkS)
       (effects (font (size 1 1) (thickness 0.15)))
     )
@@
     (fp_line (start 1 1.075) (end -1 1.075) (layer F.SilkS) (width 0.15))
     (fp_line (start -1 -1.075) (end 1 -1.075) (layer F.SilkS) (width 0.15))
-    (pad 1 smd rect (at -2 0) (size 2 1.7) (layers F.Cu F.Paste F.Mask)
+    (pad 1 smd rect (at -2 0 180) (size 2 1.7) (layers F.Cu F.Paste F.Mask)
       (net 40 "/7.4V Regulators/REG2EN"))
-    (pad 2 smd rect (at 2 0) (size 2 1.7) (layers F.Cu F.Paste F.Mask)
+    (pad 2 smd rect (at 2 0 180) (size 2 1.7) (layers F.Cu F.Paste F.Mask)
       (net 12 +12V))
     (model Resistors_SMD/R_1206_HandSoldering.wrl
@@
   )
   (module SMD_Packages:SOIC-8-N-1EP (layer F.Cu)
-    (at 109.5 -37 90)
+    (at 222.75 151.75 90)
     (descr "SO8 with exposed pad")
     (tags "SMD SO8")
@@
   )
   (gr_line (start 10.5 10.5) (end 11 10.5) (angle 90) (layer Edge.Cuts) (width 0.1))
-  (segment (start 247.75 114.75) (end 249.5 114.75) (width 0.254) (layer F.Cu) (net 2) (status 400000))
-  (segment (start 256.4 114.15) (end 258.04 114.15) (width 0.254) (layer F.Cu) (net 2) (status 800000))
+  (segment (start 247.75 114.75) (end 249.5 114.75) (width 0.254) (layer F.Cu) (net 2))
+  (segment (start 256.4 114.15) (end 258.04 114.15) (width 0.254) (layer F.Cu) (net 2))
   (segment (start 254.5 112.25) (end 256.4 114.15) (width 0.254) (layer F.Cu) (net 2))
   (segment (start 252 112.25) (end 254.5 112.25) (width 0.254) (layer F.Cu) (net 2))
@@
   (segment (start 231.583 118.083) (end 231.583 116.655) (width 0.254) (layer F.Cu) (net 12))
   (segment (start 232.25 118.75) (end 231.583 118.083) (width 0.254) (layer F.Cu) (net 12))
-  (segment (start 240.75 108.75) (end 241 108.75) (width 0.254) (layer F.Cu) (net 13) (status C00000))
-  (segment (start 241 108.75) (end 243.25 106.5) (width 0.254) (layer F.Cu) (net 13) (status 400000))
+  (segment (start 240.75 108.75) (end 241 108.75) (width 0.254) (layer F.Cu) (net 13))
+  (segment (start 241 108.75) (end 243.25 106.5) (width 0.254) (layer F.Cu) (net 13))
   (segment (start 243.25 106.5) (end 247 106.5) (width 0.254) (layer F.Cu) (net 13))
   (segment (start 247 106.5) (end 251.35 110.85) (width 0.254) (layer F.Cu) (net 13))
-  (segment (start 251.35 110.85) (end 255.5 110.85) (width 0.254) (layer F.Cu) (net 13) (status 800000))
-  (segment (start 237.27514 104.25) (end 239 104.25) (width 0.254) (layer F.Cu) (net 13) (status 400000))
-  (segment (start 240.75 106) (end 240.75 111.25) (width 0.254) (layer F.Cu) (net 13) (status 800000))
+  (segment (start 251.35 110.85) (end 255.5 110.85) (width 0.254) (layer F.Cu) (net 13))
+  (segment (start 237.27514 104.25) (end 239 104.25) (width 0.254) (layer F.Cu) (net 13))
+  (segment (start 240.75 106) (end 240.75 111.25) (width 0.254) (layer F.Cu) (net 13))
   (segment (start 239 104.25) (end 240.75 106) (width 0.254) (layer F.Cu) (net 13))
-  (segment (start 240.75 111.25) (end 240.75 113.75) (width 0.254) (layer F.Cu) (net 13) (status C00000))
-  (segment (start 240.75 113.75) (end 240.75 116.25) (width 0.254) (layer F.Cu) (net 13) (status C00000))
+  (segment (start 240.75 111.25) (end 240.75 113.75) (width 0.254) (layer F.Cu) (net 13))
+  (segment (start 240.75 113.75) (end 240.75 116.25) (width 0.254) (layer F.Cu) (net 13))
   (segment (start 236.917 115.385) (end 238.135 115.385) (width 0.254) (layer F.Cu) (net 14))
   (segment (start 242.75 112.25) (end 243.75 111.25) (width 0.254) (layer F.Cu) (net 14))
@@
   (segment (start 228.5 116.75) (end 229.865 115.385) (width 0.254) (layer F.Cu) (net 21))
   (segment (start 229.865 115.385) (end 231.583 115.385) (width 0.254) (layer F.Cu) (net 21))
-  (segment (start 231.22486 104.25) (end 230.25 104.25) (width 0.254) (layer F.Cu) (net 22) (status C00000))
-  (segment (start 230.25 104.25) (end 227.75 106.75) (width 0.254) (layer F.Cu) (net 22) (status 400000))
-  (segment (start 227.75 106.75) (end 227.75 112.75) (width 0.254) (layer F.Cu) (net 22) (status 800000))
+  (segment (start 231.22486 104.25) (end 230.25 104.25) (width 0.254) (layer F.Cu) (net 22))
+  (segment (start 230.25 104.25) (end 227.75 106.75) (width 0.254) (layer F.Cu) (net 22))
+  (segment (start 227.75 106.75) (end 227.75 112.75) (width 0.254) (layer F.Cu) (net 22))
   (segment (start 227.75 112.75) (end 228.5 112.75) (width 0.254) (layer F.Cu) (net 22))
   (segment (start 228.5 112.75) (end 229.865 114.115) (width 0.254) (layer F.Cu) (net 22))

Commit message: created a couple of different 7v4 regulator layouts
Parts:
- added C51: .1uF, Capacitors_SMD:C_1206_HandSoldering, F.Cu at (10.8, 20.6)
- moved C42 259.6 mm to (92.2, 146.2), turned to 90 degrees
- moved C46 256.6 mm to (89.8, 146.2), turned to 90 degrees
- moved R12 252.8 mm to (93.0, 154.0)
- moved R14 249.1 mm to (97.2, 148.8), turned to 180 degrees
- moved C36 245.7 mm to (93.0, 151.2)
- moved C38 240.7 mm to (97.2, 143.8), turned to 180 degrees
- moved C40 237.7 mm to (97.2, 146.2), turned to 180 degrees
- moved C45 233.2 mm to (89.8, 139.0), turned to 270 degrees
- moved L6 227.5 mm to (92.8, 130.2), turned to 180 degrees
- moved C50 226.8 mm to (92.2, 139.0), turned to 270 degrees
- moved U9 222.7 mm to (99.8, 138.0), turned to 0 degrees
- moved R16 219.1 mm to (95.0, 139.0), turned to 90 degrees
- moved C48 207.1 mm to (99.0, 129.2)
- moved C12 205.6 mm to (173.8, 35.8), turned to 0 degrees
- moved R11 204.8 mm to (181.8, 147.8), turned to 90 degrees
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Connections:
- U1 pad 1: Net-(U1-Pad1) -> /Low Voltage Regulators/REG6+3V3
- U6 pad 9: (no net) -> GND
- U7 pad 9: (no net) -> GND
- U8 pad 9: (no net) -> GND
- U9 pad 9: (no net) -> GND
Routing:
- net GND: track 29.7 -> 129.4 mm
- net /7.4V Regulators/REG3+7V4: track 0.00 -> 43.4 mm
- net /7.4V Regulators/REG4+7V4: track 0.00 -> 38.2 mm
- net /7.4V Regulators/REG2+7V4: track 0.00 -> 33.3 mm
- net +12V: track 15.9 -> 47.3 mm
- net Net-(C20-Pad2): track 0.00 -> 21.7 mm
- net Net-(C35-Pad2): track 0.00 -> 20.7 mm
- net Net-(C36-Pad2): track 0.00 -> 18.0 mm
- net Net-(C39-Pad1): track 0.00 -> 11.1 mm
- net Net-(C47-Pad2): track 0.00 -> 9.28 mm
- net Net-(C37-Pad1): track 0.00 -> 8.05 mm
- net /Servo3_PWM: track 0.00 -> 7.41 mm
- net Net-(C40-Pad1): track 0.00 -> 6.58 mm
- net Net-(C48-Pad2): track 0.00 -> 4.47 mm
- net Net-(C48-Pad1): track 0.00 -> 4.13 mm
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