File: Hardware/Arm Control Board/Arm Control Board.kicad_pcb (KiCad board)
At the start: 2 copper layers, 99 parts, among them P1 Servo 1, P10 UIM240XX_Stepper_Conn, P11 Battery, P12 SyRen, P13 Raspberry Pi, P2 Shoulder Feedback, P3 Servo 2, P4 Servo 3, P5 Elbow Feedback, P6 Servo 4, P7 RS485, P8 ST_SWD_Connector, P9 Servo 5, U1 STM32F401RCT6, U2 SN75176BDR, U3 74LVCH244APW, U4 AOZ1280CI, U5 AOZ1280CI, U6 AP65552SP-13, U7 AP65552SP-13, U8 AP65552SP-13, U9 AP65552SP-13, X1 24MHz

Commit message: Lay out regulators 1-4, update cube for oscillator
Got strangely excited about this commit. Almost called my dad...
Parts:
- added P14: Gripper Force Fdbk, MAVRIC_footprints:1x3_SMD_header, F.Cu at (228.0, 123.0)
- added R17: 20m, Resistors_SMD:R_1206_HandSoldering, F.Cu at (176.8, 154.0)
- added R18: 20m, Resistors_SMD:R_1206_HandSoldering, F.Cu at (152.5, 154.5)
- added R19: 8.06k, Resistors_SMD:R_1206_HandSoldering, F.Cu at (170.8, 160.0)
- added R20: 8.06k, Resistors_SMD:R_1206_HandSoldering, F.Cu at (146.2, 159.8)
- added R21: 20m, Resistors_SMD:R_1206_HandSoldering, F.Cu at (128.0, 154.8)
- added R22: 20m, Resistors_SMD:R_1206_HandSoldering, F.Cu at (102.8, 154.2)
- added R23: 8.06k, Resistors_SMD:R_1206_HandSoldering, F.Cu at (122.2, 160.0)
- added R24: 8.06k, Resistors_SMD:R_1206_HandSoldering, F.Cu at (97.2, 160.5)
- added U10: ZXCT1107, Housings_SOT-23_SOT-143_TSOT-6:SOT23_Transistor_Handsoldering_RevB_14Mar2014, F.Cu at (171.8, 153.2)
- added U11: ZXCT1107, Housings_SOT-23_SOT-143_TSOT-6:SOT23_Transistor_Handsoldering_RevB_14Mar2014, F.Cu at (147.0, 153.2)
- added U12: ZXCT1107, Housings_SOT-23_SOT-143_TSOT-6:SOT23_Transistor_Handsoldering_RevB_14Mar2014, F.Cu at (123.2, 153.5)
- added U13: ZXCT1107, Housings_SOT-23_SOT-143_TSOT-6:SOT23_Transistor_Handsoldering_RevB_14Mar2014, F.Cu at (98.5, 153.8)
- moved C51 186.0 mm to (175.8, 106.5)
- moved P6 5.93 mm to (102.8, 159.8), turned to 0 degrees
- moved P1 2.85 mm to (176.8, 159.2), turned to 0 degrees
- moved P4 1.50 mm to (128.0, 159.8), turned to 0 degrees
- moved P3 0.71 mm to (152.5, 159.5), turned to 0 degrees
- moved C31 0.56 mm to (181.8, 146.8)
Connections:
- net Net-(P7-Pad1) renamed /485_A
- net Net-(P7-Pad2) renamed /485_B
- C19 pad 1: /7.4V Regulators/REG1+7V4 -> Net-(C19-Pad1)
- C20 pad 1: /7.4V Regulators/REG2+7V4 -> Net-(C20-Pad1)
- C25 pad 1: /7.4V Regulators/REG1+7V4 -> Net-(C19-Pad1)
- C26 pad 1: /7.4V Regulators/REG2+7V4 -> Net-(C20-Pad1)
- C28 pad 1: /7.4V Regulators/REG1+7V4 -> Net-(C19-Pad1)
- C30 pad 1: /7.4V Regulators/REG2+7V4 -> Net-(C20-Pad1)
- C35 pad 1: /7.4V Regulators/REG3+7V4 -> Net-(C35-Pad1)
- C36 pad 1: /7.4V Regulators/REG4+7V4 -> Net-(C36-Pad1)
- C41 pad 1: /7.4V Regulators/REG3+7V4 -> Net-(C35-Pad1)
- C42 pad 1: /7.4V Regulators/REG4+7V4 -> Net-(C36-Pad1)
- C44 pad 1: /7.4V Regulators/REG3+7V4 -> Net-(C35-Pad1)
- C46 pad 1: /7.4V Regulators/REG4+7V4 -> Net-(C36-Pad1)
- L3 pad 2: /7.4V Regulators/REG1+7V4 -> Net-(C19-Pad1)
- L4 pad 2: /7.4V Regulators/REG2+7V4 -> Net-(C20-Pad1)
- L5 pad 2: /7.4V Regulators/REG3+7V4 -> Net-(C35-Pad1)
- L6 pad 2: /7.4V Regulators/REG4+7V4 -> Net-(C36-Pad1)
- R11 pad 1: /7.4V Regulators/REG3+7V4 -> Net-(C35-Pad1)
- R12 pad 1: /7.4V Regulators/REG4+7V4 -> Net-(C36-Pad1)
- R5 pad 1: /7.4V Regulators/REG1+7V4 -> Net-(C19-Pad1)
- R6 pad 1: /7.4V Regulators/REG2+7V4 -> Net-(C20-Pad1)
- U1 pad 10: GND -> Net-(U1-Pad10)
- U1 pad 11: /Low Voltage Regulators/REG6+3V3 -> Net-(U1-Pad11)
- U1 pad 12: /Low Voltage Regulators/REG6+3V3 -> GND
- U1 pad 18: (no net) -> GND
- U1 pad 20: /7.4V Regulators/REG1EN -> /7.4V Regulators/REG1CURRENT
- U1 pad 21: /7.4V Regulators/REG2EN -> /7.4V Regulators/REG2CURRENT
- U1 pad 22: /7.4V Regulators/REG3EN -> /7.4V Regulators/REG3CURRENT
- U1 pad 23: /7.4V Regulators/REG4EN -> /7.4V Regulators/REG4CURRENT
- U1 pad 27: GND -> /ADC1_IN9_Elbow
- U1 pad 33: Net-(U1-Pad33) -> /7.4V Regulators/REG1EN
- U1 pad 34: Net-(U1-Pad34) -> /7.4V Regulators/REG2EN
- U1 pad 35: Net-(U1-Pad35) -> /7.4V Regulators/REG3EN
- U1 pad 36: Net-(U1-Pad36) -> /7.4V Regulators/REG4EN
- U1 pad 54: (no net) -> Net-(U1-Pad54)
- U1 pad 55: (no net) -> Net-(U1-Pad55)
- U1 pad 8: Net-(U1-Pad8) -> /ADC1_IN10_GripForce
Routing:
- net GND: track 110.6 -> 194.6 mm, vias 5 -> 8
- net Net-(C20-Pad1): track 0.00 -> 52.2 mm
- net Net-(C19-Pad1): track 0.00 -> 51.6 mm
- net Net-(C36-Pad1): track 0.00 -> 43.9 mm
- net Net-(C35-Pad1): track 0.00 -> 41.7 mm
- net /7.4V Regulators/REG3+7V4: track 41.7 -> 0.00 mm
- net /7.4V Regulators/REG4+7V4: track 43.9 -> 3.54 mm
- net +12V: track 17.6 -> 34.9 mm
- net /7.4V Regulators/REG1EN: track 0.00 -> 11.0 mm, vias 0 -> 2
- net /7.4V Regulators/REG3EN: track 0.00 -> 10.9 mm, vias 0 -> 2
- net /7.4V Regulators/REG2EN: track 0.00 -> 10.9 mm, vias 0 -> 2
- net /7.4V Regulators/REG2+7V4: track 0.00 -> 9.92 mm
- net Net-(C31-Pad2): track 0.00 -> 9.84 mm
- net Net-(C19-Pad2): track 0.00 -> 9.25 mm
- net Net-(C32-Pad2): track 0.00 -> 9.19 mm
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- added copper zone on F.Cu, net /7.4V Regulators/REG1+7V4
- added copper zone on F.Cu, net /7.4V Regulators/REG2+7V4
- added copper zone on F.Cu, net /7.4V Regulators/REG3+7V4
- added copper zone on F.Cu, net Net-(C19-Pad1)
- added copper zone on F.Cu, net Net-(C20-Pad1)
- added copper zone on F.Cu, net Net-(C31-Pad2)
- added copper zone on F.Cu, net Net-(C32-Pad2)
- added copper zone on F.Cu, net Net-(C35-Pad1)
- added copper zone on F.Cu, net Net-(C36-Pad1)
- added copper zone on F.Cu, net Net-(C47-Pad2)

Commit message: Initial layout of Regulator 5 (AOZ)
Followed datasheet recommendations pretty well, probably some room for
improvement
Parts:
- moved D1 301.5 mm to (72.5, 139.0), turned to 270 degrees
- moved L1 288.6 mm to (67.8, 137.8)
- moved C17 194.6 mm to (78.5, 140.0), turned to 270 degrees
- moved U2 161.2 mm to (127.8, 101.0)
- moved R1 157.2 mm to (70.2, 148.2), turned to 0 degrees
- moved C13 152.6 mm to (70.2, 145.5)
- moved R2 151.9 mm to (70.2, 151.0), turned to 0 degrees
- moved U4 142.5 mm to (75.5, 139.8), turned to 0 degrees
- moved C15 141.8 mm to (70.2, 142.8), turned to 180 degrees
- moved P7 64.1 mm to (114.8, 101.8), turned to 270 degrees
- moved P13 49.7 mm to (16.0, 180.5)
- moved C51 34.8 mm to (141.5, 112.8), turned to 270 degrees
- moved U1 31.8 mm to (141.8, 101.5), turned to 270 degrees
- moved P9 15.3 mm to (63.2, 145.8), turned to 90 degrees
- moved C19 12.0 mm to (196.2, 130.5)
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Routing:
- net (no net): track 0.00 -> 15.2 mm
- net Net-(R1-Pad2): track 0.00 -> 12.0 mm
- net Net-(C15-Pad2): track 0.00 -> 10.5 mm
- net GND: track 194.6 -> 185.6 mm, vias 8 -> 3
- net /7.4V Regulators/REG2EN: track 10.9 -> 3.13 mm
- net /7.4V Regulators/REG1EN: track 11.0 -> 3.54 mm
- net /Low Voltage Regulators/REG5EN: track 0.00 -> 5.10 mm
- net Net-(C15-Pad1): track 0.00 -> 3.41 mm
- net /7.4V Regulators/REG4EN: track 11.2 -> 12.4 mm
- added copper zone on F.Cu, net /Low Voltage Regulators/REG5+5V

Commit message: Initial layout of Reg 6 (AOZ) and reorg of reg1-4
Parts:
- moved D2 290.6 mm to (72.8, 118.0), turned to 270 degrees
- moved L2 287.1 mm to (67.5, 115.8)
- moved P5 178.1 mm to (63.5, 123.8), turned to 90 degrees
- moved C14 160.3 mm to (70.5, 123.8), turned to 0 degrees
- moved R4 149.9 mm to (70.5, 129.2)
- moved R3 148.3 mm to (70.5, 126.5)
- moved C18 148.2 mm to (79.5, 118.8), turned to 270 degrees
- moved U5 144.5 mm to (76.2, 119.0), turned to 0 degrees
- moved C16 135.8 mm to (70.5, 121.2), turned to 180 degrees
- moved P8 82.9 mm to (135.5, 87.2), turned to 0 degrees
- moved R5 66.4 mm to (162.9, 185.1), turned to 0 degrees
- moved P11 63.8 mm to (94.2, 112.5), turned to 180 degrees
- moved C19 61.7 mm to (162.9, 182.4), turned to 0 degrees
- moved R9 57.5 mm to (156.9, 174.1), turned to 90 degrees
- moved R7 57.1 mm to (162.9, 179.6), turned to 180 degrees
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Routing:
- net (no net): track 15.2 -> 30.3 mm
- net Net-(C16-Pad2): track 0.00 -> 12.6 mm
- net Net-(R3-Pad2): track 0.00 -> 11.5 mm
- net /7.4V Regulators/REG4EN: track 12.4 -> 4.54 mm
- net /7.4V Regulators/REG3EN: track 10.9 -> 3.68 mm
- net /Low Voltage Regulators/REG6EN: track 0.00 -> 5.75 mm
- net Net-(C16-Pad1): track 0.00 -> 3.20 mm
- added copper zone on F.Cu, net /Low Voltage Regulators/REG6+3V3

Commit message: Continuation of board layout. 80% connected
Very poor layout so far, this will change drastically before fab
Parts:
- moved P10 155.1 mm to (116.0, 155.6), turned to 90 degrees
- moved C3 149.1 mm to (139.0, 104.8), turned to 90 degrees
- moved C4 145.1 mm to (136.2, 104.8), turned to 90 degrees
- moved C6 141.6 mm to (133.5, 104.8), turned to 90 degrees
- moved C7 138.3 mm to (130.8, 104.8), turned to 90 degrees
- moved C8 136.1 mm to (128.0, 104.8), turned to 90 degrees
- moved C11 135.4 mm to (112.5, 104.8), turned to 90 degrees
- moved C9 134.6 mm to (125.2, 104.8), turned to 90 degrees
- moved C10 133.8 mm to (122.5, 104.8), turned to 90 degrees
- moved FB1 130.0 mm to (117.5, 106.8), turned to 180 degrees
- moved P14 127.0 mm to (101.3, 131.0)
- moved P2 126.9 mm to (110.3, 131.2), turned to 0 degrees
- moved C1 124.3 mm to (136.2, 114.8), turned to 180 degrees
- moved P12 114.5 mm to (140.5, 97.2)
- moved C12 94.1 mm to (109.8, 104.8), turned to 90 degrees
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Routing:
- net /Low Voltage Regulators/REG6+3V3: track 0.00 -> 126.2 mm, vias 0 -> 4
- net /Servo5_PWM: track 0.00 -> 89.7 mm
- net /Low Voltage Regulators/REG5EN: track 5.10 -> 86.7 mm, vias 0 -> 2
- net /7.4V Regulators/REG2EN: track 3.13 -> 83.5 mm, vias 2 -> 10
- net /7.4V Regulators/REG1EN: track 3.54 -> 83.5 mm, vias 2 -> 4
- net GND: track 185.6 -> 262.5 mm, vias 3 -> 15
- net /Low Voltage Regulators/REG5+5V: track 0.00 -> 75.5 mm, vias 0 -> 2
- net /Low Voltage Regulators/REG6EN: track 5.75 -> 73.9 mm, vias 0 -> 4
- net /Servo1_PWM: track 0.00 -> 59.3 mm, vias 0 -> 2
- net /Servo2_PWM: track 0.00 -> 59.1 mm
- net /ADC1_IN10_GripForce: track 0.00 -> 56.3 mm, vias 0 -> 2
- net /Step_Direction: track 0.00 -> 53.6 mm, vias 0 -> 2
- net /ADC1_IN9_Elbow: track 0.00 -> 52.9 mm
- net /Step_Step: track 0.00 -> 52.6 mm, vias 0 -> 2
- net /Step_Enable: track 0.00 -> 52.0 mm, vias 0 -> 2
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
Commit message: Reorganize all regulators. Reorganize buffer pins
Pins reorganized to simplify board flow
Parts:
- moved R4 170.0 mm to (252.1, 77.6), turned to 90 degrees
- moved R3 164.9 mm to (249.3, 77.6), turned to 90 degrees
- moved C14 159.9 mm to (246.6, 77.6), turned to 90 degrees
- moved C18 159.7 mm to (241.6, 68.6), turned to 0 degrees
- moved U5 156.8 mm to (241.8, 71.8), turned to 90 degrees
- moved C16 155.4 mm to (244.1, 77.6), turned to 270 degrees
- moved P5 154.6 mm to (246.6, 84.6), turned to 180 degrees
- moved R5 151.8 mm to (170.2, 33.5), turned to 180 degrees
- moved D2 151.6 mm to (240.8, 75.3), turned to 0 degrees
- moved P14 150.7 mm to (246.6, 91.1), turned to 180 degrees
- moved C19 146.3 mm to (170.2, 36.2), turned to 180 degrees
- moved C21 145.1 mm to (165.2, 36.8), turned to 90 degrees
- moved L2 142.9 mm to (238.6, 80.6), turned to 90 degrees
- moved R20 142.6 mm to (215.2, 31.5), turned to 0 degrees
- moved R7 140.8 mm to (170.2, 39.0), turned to 0 degrees
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Connections:
- U3 pad 11: /GPIO_PB9_Enable -> /TIM4_CH1_EE
- U3 pad 12: /Servo4_PWM -> /Servo1_PWM
- U3 pad 13: /GPIO_PB8_Direction -> /TIM4_CH2_Step
- U3 pad 14: /Servo3_PWM -> /Servo2_PWM
- U3 pad 15: /TIM4_CH2_Step -> /GPIO_PB8_Direction
- U3 pad 16: /Servo2_PWM -> /Servo3_PWM
- U3 pad 17: /TIM4_CH1_EE -> /GPIO_PB9_Enable
- U3 pad 18: /Servo1_PWM -> /Servo4_PWM
- U3 pad 2: /TIM3_CH1_EE -> /TIM3_CH4_EE
- U3 pad 3: /Servo5_PWM -> /Step_Enable
- U3 pad 4: /TIM3_CH2_EE -> /TIM3_CH3_EE
- U3 pad 5: /Step_Step -> /Step_Direction
- U3 pad 6: /TIM3_CH3_EE -> /TIM3_CH2_EE
- U3 pad 7: /Step_Direction -> /Step_Step
- U3 pad 8: /TIM3_CH4_EE -> /TIM3_CH1_EE
- U3 pad 9: /Step_Enable -> /Servo5_PWM
Routing:
- net /Servo5_PWM: track 89.7 -> 0.00 mm
- net /Low Voltage Regulators/REG5EN: track 86.7 -> 0.22 mm, vias 2 -> 0
- net /7.4V Regulators/REG2EN: track 83.5 -> 0.00 mm, vias 10 -> 0
- net /7.4V Regulators/REG1EN: track 83.5 -> 0.01 mm, vias 4 -> 0
- net /Low Voltage Regulators/REG5+5V: track 75.5 -> 0.00 mm, vias 2 -> 0
- net /Low Voltage Regulators/REG6EN: track 73.9 -> 0.47 mm, vias 4 -> 0
- net /Servo1_PWM: track 59.3 -> 0.00 mm, vias 2 -> 0
- net /Servo2_PWM: track 59.1 -> 0.00 mm
- net /ADC1_IN10_GripForce: track 56.3 -> 0.00 mm, vias 2 -> 0
- net /ADC1_IN9_Elbow: track 52.9 -> 0.00 mm
- net /Step_Step: track 52.6 -> 0.00 mm, vias 2 -> 0
- net /Servo4_PWM: track 48.4 -> 0.00 mm, vias 2 -> 0
- net /ADC1_IN8_Shoulder: track 45.1 -> 0.21 mm, vias 2 -> 0
- net /Servo3_PWM: track 40.6 -> 0.00 mm, vias 2 -> 0
- net GND: track 262.5 -> 222.6 mm, vias 15 -> 4
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- removed copper zone on B.Cu, net GND
